Commit message: 修复了少量变量bug，已在ROS2 Humble上完成运行

File: RGS_DRL/src/agent_description/urdf/ackerman.xacro (robot description, xacro)
@@ -196,5 +196,5 @@
         <plugin filename="libgazebo_ros2_control.so" name="gazebo_ros2_control">
             <!-- /{controller_name}/commands -->
-            <parameters>$(find agent_description)/config/MAV_controller.yaml</parameters>
+            <parameters>$(find agent_description)/config/ackerman_controller.yaml</parameters>
         </plugin>
     </gazebo>

File: RGS_DRL/src/agent_description/urdf/differential.urdf (robot description, URDF)
Before this commit: robot differential, 8 links, 7 joints
Joints:
- joint lidar_joint: origin xyz=-0.1 0.0 0.05 rpy=0.0 0.0 0.0 -> xyz=-0.1 0.0 0.05 rpy=0.0 0.0 3.1416
